File: PCB_Micro/esp32_fpga/_autosave-esp32_fpga.kicad_sch (KiCad schematic)
At the start: 86 parts, among them IC1 ICE40UP5K-SG48I, J1 DM3AT-SF-PEJM5, J3 USB_C_Receptacle_USB2.0_16P, J4 Conn_01x04_Pin, J5 AUX1, J6 AUX2, Q1 DMP1045U-7, SW1 SW_Push, U1 ESP32-S3-WROOM-1-N8R8, U2 BME280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

Commit message: schématique complet
Parts:
- added R17: 10k, Resistor_SMD:R_0603_1608Metric, symbol Device:R
- D3: value LED -> LED Green
Connections:
- net GND: now also R17.2
- net VBUS: now also R17.1
Changed lines of the file:
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@@
 	)
 	(junction
+		(at 85.09 170.18)
+		(diameter 0)
+		(color 0 0 0 0)
+	)
+	(junction
 		(at 82.55 246.38)
 		(diameter 0)
@@
 	)
 	(junction
+		(at 26.67 160.02)
+		(diameter 0)
+		(color 0 0 0 0)
+	)
+	(junction
 		(at 48.26 246.38)
 		(diameter 0)
@@
 	(wire
 		(pts
+			(xy 85.09 170.18) (xy 88.9 170.18)
+		)
+		(stroke
+			(width 0)
+			(type default)
+		)
+	)
+	(wire
+		(pts
 			(xy 172.72 46.99) (xy 177.8 46.99)
 		)
@@
 	(wire
 		(pts
-			(xy 34.29 92.71) (xy 17.145 92.71)
-		)
-		(stroke
-			(width 0)
-			(type default)
-		)
-	)
-	(wire
-		(pts
 			(xy 43.18 213.36) (xy 43.18 215.9)
 		)
@@
 	(wire
 		(pts
-			(xy 53.34 121.92) (xy 53.34 134.62)
-		)
-		(stroke
-			(width 0)
-			(type default)
-		)
-	)
-	(wire
-		(pts
 			(xy 278.13 212.09) (xy 278.13 227.33)
 		)
@@
 	(wire
 		(pts
-			(xy 34.29 59.69) (xy 17.145 59.69)
-		)
-		(stroke
-			(width 0)
-			(type default)
-		)
-	)
-	(wire
-		(pts
 			(xy 344.17 110.49) (xy 344.17 104.14)
 		)
@@
 	(wire
 		(pts
+			(xy 19.05 160.02) (xy 26.67 160.02)
+		)
+		(stroke
+			(width 0)
+			(type default)
+		)
+	)
+	(wire
+		(pts
 			(xy 264.16 74.93) (xy 264.16 83.82)
 		)
@@
 	(wire
 		(pts
+			(xy 85.09 170.18) (xy 85.09 181.61)
+		)
+		(stroke
+			(width 0)
+			(type default)
+		)
+	)
+	(wire
+		(pts
 			(xy 227.33 163.83) (xy 267.97 163.83)
 		)
@@
 	(wire
 		(pts
-			(xy 34.29 95.25) (xy 17.145 95.25)
+			(xy 335.28 26.67) (xy 330.2 26.67)
 		)
 		(stroke
@@
 	(wire
 		(pts
-			(xy 335.28 26.67) (xy 330.2 26.67)
+			(xy 281.94 74.93) (xy 281.94 83.82)
 		)
 		(stroke
@@
 	(wire
 		(pts
-			(xy 281.94 74.93) (xy 281.94 83.82)
+			(xy 49.53 24.13) (xy 34.29 24.13)
 		)
 		(stroke
@@
 	(wire
 		(pts
-			(xy 49.53 24.13) (xy 34.29 24.13)
+			(xy 53.34 121.92) (xy 53.34 132.08)
 		)
 		(stroke
@@
 	(wire
 		(pts
-			(xy 229.87 246.38) (xy 237.49 246.38)
-		)
-		(stroke
-			(width 0)
-			(type default)
-		)
-	)
-	(wire
-		(pts
 			(xy 238.76 250.19) (xy 234.95 250.19)
 		)
@@
 	(wire
 		(pts
+			(xy 17.78 87.63) (xy 34.29 87.63)
+		)
+		(stroke
+			(width 0)
+			(type default)
+		)
+	)
+	(wire
+		(pts
 			(xy 38.1 121.92) (xy 38.1 129.54)
 		)
@@
 	(wire
 		(pts
+			(xy 17.78 59.69) (xy 34.29 59.69)
+		)
+		(stroke
+			(width 0)
+			(type default)
+		)
+	)
+	(wire
+		(pts
 			(xy 300.99 74.93) (xy 300.99 81.28)
 		)
@@
 	(wire
 		(pts
+			(xy 17.78 92.71) (xy 34.29 92.71)
+		)
+		(stroke
+			(width 0)
+			(type default)
+		)
+	)
+	(wire
+		(pts
 			(xy 280.67 125.73) (xy 280.67 130.81)
 		)
@@
 	(wire
 		(pts
-			(xy 34.29 69.85) (xy 17.145 69.85)
+			(xy 397.51 49.53) (xy 398.78 49.53)
 		)
 		(stroke
@@
 	(wire
 		(pts
-			(xy 397.51 49.53) (xy 398.78 49.53)
+			(xy 17.78 85.09) (xy 34.29 85.09)
 		)
 		(stroke
@@
 	(wire
 		(pts
-			(xy 16.51 67.31) (xy 34.29 67.31)
-		)
-		(stroke
-			(width 0)
-			(type default)
-		)
-	)
-	(wire
-		(pts
 			(xy 405.13 30.48) (xy 405.13 31.75)
 		)
@@
 	(wire
 		(pts
-			(xy 34.29 85.09) (xy 17.145 85.09)
-		)
-		(stroke
-			(width 0)
-			(type default)
-		)
-	)
-	(wire
-		(pts
 			(xy 377.19 176.53) (xy 377.19 181.61)
 		)
@@
 	(wire
 		(pts
+			(xy 17.78 95.25) (xy 34.29 95.25)
+		)
+		(stroke
+			(width 0)
+			(type default)
+		)
+	)
+	(wire
+		(pts
 			(xy 406.4 110.49) (xy 406.4 104.14)
 		)
@@
 	(wire
 		(pts
-			(xy 34.29 87.63) (xy 17.145 87.63)
-		)
-		(stroke
-			(width 0)
-			(type default)
-		)
-	)
-	(wire
-		(pts
 			(xy 214.63 86.36) (xy 214.63 82.55)
 		)
@@
 	(wire
 		(pts
-			(xy 74.93 170.18) (xy 88.9 170.18)
+			(xy 74.93 170.18) (xy 85.09 170.18)
 		)
 		(stroke
@@
 	(wire
 		(pts
+			(xy 17.78 69.85) (xy 34.29 69.85)
+		)
+		(stroke
+			(width 0)
+			(type default)
+		)
+	)
+	(wire
+		(pts
 			(xy 397.51 39.37) (xy 407.67 39.37)
 		)
@@
 	(wire
 		(pts
+			(xy 17.78 67.31) (xy 34.29 67.31)
+		)
+		(stroke
+			(width 0)
+			(type default)
+		)
+	)
+	(wire
+		(pts
 			(xy 22.86 121.92) (xy 22.86 133.35)
 		)
@@
 		)
 	)
-	(label "VBAT"
-		(at 237.49 246.38 0)
-		(effects
-			(font
-				(size 1.524 1.524)
-			)
-			(justify left bottom)
-		)
-	)
 	(label "FPGA_P2"
 		(at 248.92 156.21 180)
@@
 	)
 	(label "ADC"
-		(at 229.87 246.38 180)
+		(at 85.09 181.61 270)
 		(effects
 			(font
@@
 	)
 	(symbol
+		(lib_id "power:GND")
+		(at 19.05 167.64 0)
+		(unit 1)
+		(exclude_from_sim no)
+		(in_bom yes)
+		(on_board yes)
+		(dnp no)
+		(property "Reference" "#PWR038"
+			(at 19.05 173.99 0)
+			(effects
+				(font
+					(size 1.27 1.27)
+				)
+				(hide yes)
+			)
+		)
+		(property "Value" "GND"
+			(at 19.05 171.45 0)
+			(effects
+				(font
+					(size 1.27 1.27)
+				)
+			)
+		)
+		(property "Footprint" ""
+			(at 19.05 167.64 0)
+			(effects
+				(font
+					(size 1.27 1.27)
+				)
+			)
+		)
+		(property "Datasheet" ""
+			(at 19.05 167.64 0)
+			(effects
+				(font
+					(size 1.27 1.27)
+				)
+			)
+		)
+		(property "Description" ""
+			(at 19.05 167.64 0)
+			(effects
+				(font
+					(size 1.27 1.27)
+				)
+			)
+		)
+		(pin "1"
+		)
+		(instances
+			(project "esp32_fpga"
+				(path "/e9b45eef-13aa-420c-803d-e39bf82057f5"
+					(reference "#PWR038")
+					(unit 1)
+				)
+			)
+		)
+	)
+	(symbol
 		(lib_id "Device:R_Pack04")
 		(at 394.97 99.06 0)
@@
 			)
 		)
-		(property "Value" "LED"
+		(property "Value" "LED Green"
 			(at 408.94 208.5974 90)
 			(effects
@@
 					(unit 1)
 				)
+			)
+		)
+	)
+	(symbol
+		(lib_id "Device:R")
+		(at 19.05 163.83 0)
+		(unit 1)
+		(exclude_from_sim no)
+		(in_bom yes)
+		(on_board yes)
+		(dnp no)
+		(property "Reference" "R17"
+			(at 21.082 163.83 90)
+			(effects
+				(font
+					(size 1.27 1.27)
+				)
+			)
+		)
+		(property "Value" "10k"
+			(at 19.05 163.83 90)
+			(effects
+				(font
+					(size 1.27 1.27)
+				)
+			)
+		)
+		(property "Footprint" "Resistor_SMD:R_0603_1608Metric"
+			(at 17.272 163.83 0)
+			(effects
+				(font
+					(size 1.27 1.27)
+				)
+				(hide yes)
+			)
+		)
+		(property "Datasheet" ""
+			(at 19.05 163.83 0)
+			(effects
+				(font
+					(size 1.27 1.27)
+				)
+			)
+		)
+		(property "Description" ""
+			(at 19.05 163.83 0)
+			(effects
+				(font
+					(size 1.27 1.27)
+				)
+			)
+		)
+		(pin "1"
+		)
+		(pin "2"
+		)
+		(instances
+			(project "esp32_fpga"
+				(path "/e9b45eef-13aa-420c-803d-e39bf82057f5"
+					(reference "R17")
+					(unit 1)
+				)

Commit message: Début PCB
Parts:
- removed J5: AUX1, Connector_PinSocket_2.00mm:PinSocket_1x19_P2.00mm_Vertical, symbol Connector_Generic:Conn_01x19
- removed J6: AUX2, Connector_PinSocket_2.00mm:PinSocket_1x19_P2.00mm_Vertical, symbol Connector_Generic:Conn_01x19
- added J2: AUX1, Connector_PinSocket_1.00mm:PinSocket_1x14_P1.00mm_Vertical, symbol Connector_Generic:Conn_01x14
- added J7: AUX2, Connector_PinSocket_1.27mm:PinSocket_1x08_P1.27mm_Vertical, symbol Connector_Generic:Conn_01x08
- added J8: AUX3, Connector_PinSocket_1.00mm:PinSocket_1x14_P1.00mm_Vertical, symbol Connector_Generic:Conn_01x14
Connections:
- net +3.3V: now also J2.2 (Pin_2)
- net FPGA_P34: now also J2.4 (Pin_4)
- net GND: now also J2.1 (Pin_1), J8.1 (Pin_1)
- net GPIO0: now also J8.14 (Pin_14)
- net GPIO1: now also J8.2 (Pin_2)
- net GPIO14: now also J7.4 (Pin_4)
- net GPIO17: now also J2.10 (Pin_10)
- net GPIO18: now also J2.11 (Pin_11)
- net GPIO2: now also J8.3 (Pin_3)
- net GPIO21: now also J7.5 (Pin_5)
- net GPIO3: now also J7.1 (Pin_1)
- net GPIO38: now also J8.10 (Pin_10)
- net GPIO40: now also J8.8 (Pin_8)
- net GPIO41: now also J8.7 (Pin_7)
- net GPIO42: now also J8.6 (Pin_6)
- net GPIO47: now also J7.6 (Pin_6)
- net GPIO48: now also J7.7 (Pin_7)
- net GPIO5: now also J2.7 (Pin_7)
- net GPIO6: now also J2.8 (Pin_8)
- net GPIO7: now also J2.9 (Pin_9)
- net GPIO8: now also J2.12 (Pin_12)
- net GPIO9: now also J7.3 (Pin_3)
- net NRST: now also J2.3 (Pin_3)
- net SCL: now also J7.2 (Pin_2)
- net SDA: now also J7.8 (Pin_8)
- net SPI2_CLK: now also J8.12 (Pin_12)
- net SPI2_CS: now also J8.9 (Pin_9)
- net SPI2_MISO: now also J8.11 (Pin_11)
- net SPI2_MOSI: now also J8.13 (Pin_13)
- net UART_RX: now also J8.5 (Pin_5)
- net UART_TX: now also J8.4 (Pin_4)
- net USB D+: now also J2.14 (Pin_14)
- net USB D-: now also J2.13 (Pin_13)
- no-connect marks 6 -> 8
