File: PCB_Micro/esp32_fpga/esp32_fpga.kicad_pcb (KiCad board)
At the start: 2 copper layers, 88 parts, among them IC1 ICE40UP5K-SG48I, J1 DM3AT-SF-PEJM5, J2 AUX1, J3 USB_C_Receptacle_USB2.0_16P, J4 Conn_01x04_Pin, J5 AUX2, J8 AUX3, Q1 DMP1045U-7, SW1 SW_Push, U1 ESP32-S3-WROOM-1-N8R8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

Commit message: PCB presque terminé
Parts:
- J4: footprint Connector:NS-Tech_Grove_1x04_P2mm_Vertical -> Connector_PinHeader_2.00mm:PinHeader_1x04_P2.00mm_Vertical_SMD_Pin1Left
- J5: moved to B.Cu
- TP1, TP2, TP3, TP4: footprint TestPoint:TestPoint_Pad_D1.0mm -> TestPoint:TestPoint_THTPad_1.0x1.0mm_Drill0.5mm
- moved MK2 145.3 mm to (166.6, 121.1), turned to 180 degrees
- moved C4 118.9 mm to (125.3, 49.3)
- moved R4 114.5 mm to (127.0, 48.0), turned to 0 degrees
- moved MK1 95.3 mm to (126.2, 52.0), turned to 0 degrees
- moved D3 93.7 mm to (139.0, 67.6), turned to -90 degrees
- moved C31 92.3 mm to (114.1, 117.6), turned to 180 degrees
- moved R14 91.0 mm to (139.7, 70.6), turned to -90 degrees
- moved J1 89.2 mm to (128.5, 62.8), turned to 119.696 degrees
- moved TP8 87.1 mm to (123.7, 121.8)
- moved C6 85.1 mm to (87.3, 122.2), turned to 0 degrees
- moved C30 81.4 mm to (110.5, 74.2)
- moved PMOD1 81.1 mm to (115.6, 84.6)
- moved U5 79.5 mm to (100.1, 105.2)
- moved J4 78.7 mm to (122.7, 79.9), turned to -90 degrees
- moved U6 78.0 mm to (117.7, 101.0), turned to -90 degrees
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Connections:
- MK1 pad 1: /PIN_P2 -> /PIN_P6
- MK1 pad 2: /PIN_P3 -> /PIN_P9
- MK1 pad 3: /PIN_P4 -> /PIN_P10
Routing:
- net GND: track 0.00 -> 129.6 mm, vias 0 -> 48
- net +3.3V: track 0.00 -> 100.7 mm, vias 0 -> 38
- net /PIN_P20: track 0.00 -> 60.2 mm, vias 0 -> 1
- net +4V: track 0.00 -> 58.1 mm, vias 0 -> 4
- net /PIN_P18: track 0.00 -> 58.1 mm, vias 0 -> 1
- net /PIN_P19: track 0.00 -> 56.1 mm, vias 0 -> 1
- net /CDONE: track 0.00 -> 49.7 mm, vias 0 -> 2
- net Net-(U3-PWRGD): track 0.00 -> 47.9 mm, vias 0 -> 4
- net /CRESET: track 0.00 -> 47.5 mm, vias 0 -> 2
- net +1V2: track 0.00 -> 35.0 mm, vias 0 -> 2
- net /~{PSRAM_CS}: track 0.00 -> 29.2 mm, vias 0 -> 2
- net /VBUS: track 0.00 -> 29.1 mm
- net /SPI_MISO: track 0.00 -> 29.0 mm
- net /SPI_CLK: track 0.00 -> 28.2 mm
- net /SPI_MOSI: track 0.00 -> 27.6 mm
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- added copper zone on In2.Cu, net +3.3V
- added copper zone on In1.Cu, net GND
Other:
- board outline added: 92.8 x 79.5 mm
- copper layers 2 -> 4

Commit message: PCB rooté reste les erreurs a voir
Parts:
- removed J1: DM3AT-SF-PEJM5, custom:HRS_DM3AT-SF-PEJM5
- removed TP1: SPI_MISO, TestPoint:TestPoint_THTPad_1.0x1.0mm_Drill0.5mm
- removed TP2: SPI_CLK, TestPoint:TestPoint_THTPad_1.0x1.0mm_Drill0.5mm
- removed TP3: SPI_CS, TestPoint:TestPoint_THTPad_1.0x1.0mm_Drill0.5mm
- removed TP4: SPI_MOSI, TestPoint:TestPoint_THTPad_1.0x1.0mm_Drill0.5mm
- removed TP5: CDONE, TestPoint:TestPoint_Pad_D1.0mm
- removed TP6: CRESET, TestPoint:TestPoint_Pad_D1.0mm
- added D8: LED_RGB, LED_SMD:LED_RGB_5050-6, B.Cu at (127.9, 62.3)
- added J6: 503398-1892, custom:5033981892, F.Cu at (133.6, 68.7)
- added kibuzzard-628C6D93: G***, kibuzzard-628C6D93, F.Cu at (110.6, 149.6)
- moved J5 8.40 mm to (133.4, 96.6), turned to 28 degrees
- moved U1 8.18 mm to (144.7, 84.9), turned to 118 degrees
- moved J2 6.48 mm to (152.5, 94.1), turned to 118 degrees
- moved J8 5.72 mm to (142.3, 73.0), turned to 118 degrees
- moved C13 4.34 mm to (155.3, 94.5), turned to -90 degrees
- moved C9 3.27 mm to (155.6, 97.7), turned to 0 degrees
- moved RN2 2.84 mm to (108.8, 89.4)
- moved C3 2.22 mm to (152.2, 103.3)
- moved R3 2.22 mm to (155.2, 103.7)
- moved SW1 2.22 mm to (155.2, 100.8)
- moved C11 1.97 mm to (121.5, 70.3), turned to 180 degrees
- moved D3 1.96 mm to (138.4, 65.7)
- moved R14 1.96 mm to (139.2, 68.7)
Connections:
- IC1 pad 34: /FPGA_P34 -> unconnected-(IC1-IOT_44B-Pad34)
- J2 pad 4: /FPGA_P34 -> /ADC
- J2 pad 5: unconnected-(J2-Pin_5-Pad5) -> /GPIO5
- J2 pad 6: unconnected-(J2-Pin_6-Pad6) -> /GPIO6
- J2 pad 7: /GPIO5 -> /GPIO7
- J2 pad 8: /GPIO6 -> /CDONE
- J2 pad 9: /GPIO7 -> /CRESET
- U1 pad 41_10: (no net) -> GND
- U1 pad 41_11: (no net) -> GND
- U1 pad 41_12: (no net) -> GND
- U1 pad 41_13: (no net) -> GND
- U1 pad 41_14: (no net) -> GND
- U1 pad 41_15: (no net) -> GND
- U1 pad 41_16: (no net) -> GND
- U1 pad 41_17: (no net) -> GND
- U1 pad 41_18: (no net) -> GND
- U1 pad 41_19: (no net) -> GND
- U1 pad 41_20: (no net) -> GND
- U1 pad 41_21: (no net) -> GND
Routing:
- net /PIN_P6: track 18.2 -> 50.5 mm
- net GND: track 129.6 -> 159.7 mm, vias 48 -> 73
- net /PIN_P18: track 58.1 -> 87.0 mm, vias 1 -> 4
- net /PIN_P19: track 56.1 -> 84.9 mm, vias 1 -> 2
- net /PIN_P10: track 14.1 -> 42.8 mm, vias 0 -> 1
- net /PIN_P2: track 0.00 -> 27.6 mm, vias 0 -> 1
- net Net-(D1-BK): track 0.00 -> 26.4 mm, vias 0 -> 2
- net /PIN_P46: track 7.33 -> 33.2 mm, vias 0 -> 1
- net /PIN_P43: track 0.00 -> 25.8 mm
- net /PIN_P9: track 18.8 -> 44.4 mm, vias 0 -> 1
- net /PIN_P4: track 0.00 -> 24.2 mm, vias 0 -> 1
- net /SCL: track 4.55 -> 27.1 mm, vias 0 -> 1
- net /PIN_P3: track 0.00 -> 21.9 mm, vias 0 -> 1
- net /PIN_P13: track 0.00 -> 21.8 mm, vias 0 -> 1
- net /ADC: track 26.2 -> 47.5 mm
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Other:
- board size 92.8 x 79.5 mm -> 92.8 x 79.4 mm
- board text added: "(+)"
- board text added: "(-)"
- board text added: "3v3"
- board text added: "4v"
- board text added: "BOOT"
- board text added: "C3 LED"
- board text added: "C3 USB PWR"
- board text added: "CHG"
- board text added: "DONE"
- board text added: "LiPo"
- board text added: "PWR"
- board text added: "RGB"
- board text added: "RST"

Commit message: PCB terminé avec gerber sans LEDs niveau sonore
Parts:
- removed D8: LED_RGB, LED_SMD:LED_RGB_5050-6
- added SW2: SW_Push, Button_Switch_SMD:SW_SPST_PTS810, B.Cu at (124.3, 74.7)
Routing:
- net /GPIO0: track 3.37 -> 14.9 mm
- net GND: track 159.7 -> 163.8 mm, vias 73 -> 74

Commit message: Ajout de labels et modifications d'empreinte tjr sans LED
Parts:
- removed kibuzzard-628C6D93: G***, kibuzzard-628C6D93
- J4: footprint Connector_PinHeader_2.00mm:PinHeader_1x04_P2.00mm_Vertical_SMD_Pin1Left -> Connector_PinSocket_2.54mm:PinSocket_1x04_P2.54mm_Vertical
- PMOD1, PMOD2, PMOD3: footprint Connector_PinSocket_2.54mm:PinSocket_2x06_P2.54mm_Vertical -> Connector_Samtec_HLE_THT:Samtec_HLE-106-02-xx-DV-TE_2x06_P2.54mm_Horizontal
- moved J4 3.24 mm to (119.4, 79.9)
- turned PMOD1 to 90 degrees
- turned PMOD2 to -90 degrees
- turned PMOD3 to 0 degrees
Routing:
- net /SCL: track 27.1 -> 26.3 mm
Other:
- board text added: "+"
- board text added: "-"
- board text added: "ECAM Davidson-Hugo-Adam-Matthieu"
- board text added: "USB_PWR"
- board text removed: "(+)"
- board text removed: "(-)"
- board text removed: "3v3"
- board text removed: "4v"
- board text removed: "C3 LED"
- board text removed: "C3 USB PWR"
- board text removed: "CHG"
- board text removed: "DONE"
- board text removed: "LiPo"
- board text removed: "PWR"
- board text removed: "RGB"

Commit message: PCB et schématique modifié pour l'implémentation de la LED RGB avec alim externe
Parts:
- added BT2: Battery Connector, Connector_JST:JST_EH_B2B-EH-A_1x02_P2.50mm_Vertical, B.Cu at (115.7, 63.5)
- added C12: 0.1uf, Capacitor_SMD:C_0402_1005Metric, B.Cu at (122.0, 59.7)
- added C14: 47uf 10V, Capacitor_SMD:C_0402_1005Metric, B.Cu at (120.6, 61.2)
- added D8: LED_RGB, LED_SMD:LED_RGB_5050-6, B.Cu at (127.3, 62.8)
- added Q2: BSS138, Package_TO_SOT_SMD:SOT-23, B.Cu at (130.7, 57.3)
- added Q3: BSS138, Package_TO_SOT_SMD:SOT-23, B.Cu at (136.2, 60.9)
- added Q4: BSS138, Package_TO_SOT_SMD:SOT-23, B.Cu at (134.3, 65.0)
- added R18: 10k, Resistor_SMD:R_0603_1608Metric, B.Cu at (131.9, 52.7)
- added R19: 10k, Resistor_SMD:R_0603_1608Metric, B.Cu at (138.2, 63.4)
- added R20: 10k, Resistor_SMD:R_0603_1608Metric, B.Cu at (137.3, 68.0)
- added R21: 150, Resistor_SMD:R_0603_1608Metric, B.Cu at (124.0, 55.9)
- added R22: 100, Resistor_SMD:R_0603_1608Metric, B.Cu at (132.6, 61.0)
- added R23: 100, Resistor_SMD:R_0603_1608Metric, B.Cu at (131.6, 67.1)
Routing:
- net /GPIO40: track 3.10 -> 31.9 mm, vias 0 -> 1
- net /GPIO41: track 3.07 -> 22.2 mm, vias 0 -> 1
- net Net-(BT2-Pin_1): track 0.00 -> 16.2 mm, vias 0 -> 2
- net GND: track 163.9 -> 177.6 mm, vias 74 -> 82
- net /GPIO42: track 3.05 -> 15.7 mm
- net Net-(D8-RK): track 0.00 -> 9.86 mm, vias 0 -> 2
- net Net-(Q2-D): track 0.00 -> 6.44 mm, vias 0 -> 2
- net Net-(D8-GK): track 0.00 -> 4.15 mm
- net Net-(Q4-D): track 0.00 -> 3.74 mm
- net Net-(Q3-D): track 0.00 -> 3.07 mm
- net Net-(D8-BK): track 0.00 -> 2.59 mm
Other:
- board text added: "+5"
- board text added: "BAT+"
- board text added: "PWR_LED"
- board text removed: "+"
